Commit message: Initial commit

File: src/aries/urdf/aries_gazebo.xacro (robot description, xacro)
@@ -113,5 +113,8 @@
             <joint_name>arm_shoulder_joint</joint_name>
             <joint_name>arm_elbow_joint</joint_name>
-            <joint_name>arm_gripper_joint</joint_name>
+            <joint_name>arm_wrist_joint</joint_name>
+            <joint_name>arm_gripper_base_joint</joint_name>
+            <joint_name>arm_gripper_left_joint</joint_name>
+            <joint_name>arm_gripper_right_joint</joint_name>
             <joint_name>L_Rocker_Joint</joint_name>
             <joint_name>R_Rocker_Joint</joint_name>
@@ -145,5 +148,5 @@
       <i_min>-6</i_min><i_max>6</i_max>
     </plugin>
-    <plugin filename="gz-sim-joint-position-controller-system"
+    <!-- <plugin filename="gz-sim-joint-position-controller-system"
         name="gz::sim::systems::JointPositionController">
       <joint_name>L_Boggie_Joint</joint_name>
@@ -154,9 +157,10 @@
       <joint_name>R_Boggie_Joint</joint_name>
       <topic>/model/aries/joint/R_Boggie_Joint/cmd_pos</topic>
-    </plugin>
+    </plugin> -->
     <plugin filename="gz-sim-joint-position-controller-system"
         name="gz::sim::systems::JointPositionController">
       <joint_name>arm_base_joint</joint_name>
       <topic>/model/aries/joint/arm_base_joint/cmd_pos</topic>
+      <initial_position>0.0</initial_position>
       <p_gain>300</p_gain><i_gain>2</i_gain><d_gain>30</d_gain>
       <i_min>-6</i_min><i_max>6</i_max>
@@ -166,4 +170,5 @@
       <joint_name>arm_shoulder_joint</joint_name>
       <topic>/model/aries/joint/arm_shoulder_joint/cmd_pos</topic>
+      <initial_position>0.510</initial_position>
       <p_gain>300</p_gain><i_gain>2</i_gain><d_gain>30</d_gain>
       <i_min>-6</i_min><i_max>6</i_max>
@@ -173,11 +178,37 @@
       <joint_name>arm_elbow_joint</joint_name>
       <topic>/model/aries/joint/arm_elbow_joint/cmd_pos</topic>
-      <p_gain>300</p_gain><i_gain>2</i_gain><d_gain>30</d_gain>
-      <i_min>-6</i_min><i_max>6</i_max>
-    </plugin>
-    <plugin filename="gz-sim-joint-position-controller-system"
-        name="gz::sim::systems::JointPositionController">
-      <joint_name>arm_gripper_joint</joint_name>
-      <topic>/model/aries/joint/arm_gripper_joint/cmd_pos</topic>
+      <initial_position>1.748</initial_position>
+      <p_gain>300</p_gain><i_gain>2</i_gain><d_gain>30</d_gain>
+      <i_min>-6</i_min><i_max>6</i_max>
+    </plugin>
+    <plugin filename="gz-sim-joint-position-controller-system"
+        name="gz::sim::systems::JointPositionController">
+      <joint_name>arm_wrist_joint</joint_name>
+      <topic>/model/aries/joint/arm_wrist_joint/cmd_pos</topic>
+      <initial_position>1.420</initial_position>
+      <p_gain>300</p_gain><i_gain>2</i_gain><d_gain>30</d_gain>
+      <i_min>-6</i_min><i_max>6</i_max>
+    </plugin>
+    <plugin filename="gz-sim-joint-position-controller-system"
+        name="gz::sim::systems::JointPositionController">
+      <joint_name>arm_gripper_base_joint</joint_name>
+      <topic>/model/aries/joint/arm_gripper_base_joint/cmd_pos</topic>
+      <initial_position>0.0</initial_position>
+      <p_gain>300</p_gain><i_gain>2</i_gain><d_gain>30</d_gain>
+      <i_min>-6</i_min><i_max>6</i_max>
+    </plugin>
+    <plugin filename="gz-sim-joint-position-controller-system"
+        name="gz::sim::systems::JointPositionController">
+      <joint_name>arm_gripper_left_joint</joint_name>
+      <topic>/model/aries/joint/arm_gripper_left_joint/cmd_pos</topic>
+      <initial_position>0.0</initial_position>
+      <p_gain>300</p_gain><i_gain>2</i_gain><d_gain>30</d_gain>
+      <i_min>-6</i_min><i_max>6</i_max>
+    </plugin>
+    <plugin filename="gz-sim-joint-position-controller-system"
+        name="gz::sim::systems::JointPositionController">
+      <joint_name>arm_gripper_right_joint</joint_name>
+      <topic>/model/aries/joint/arm_gripper_right_joint/cmd_pos</topic>
+      <initial_position>0.0</initial_position>
       <p_gain>300</p_gain><i_gain>2</i_gain><d_gain>30</d_gain>
       <i_min>-6</i_min><i_max>6</i_max>

File: src/aries/urdf/arm.xacro (robot description, xacro)
@@ -129,38 +129,39 @@
         <dynamics damping="10" friction="2"/>
     </joint>
-    <link name="arm_gripper_link">
-        <inertial>
-            <origin xyz="0 0 0" rpy="0 0 0" />
-            <mass value="1.5363204791731" />
-            <inertia
-                ixx="0.242660790998556"
-                ixy="-9.00009815481889E-05"
-                ixz="0.0234683038167963"
-                iyy="0.514730499629884"
-                iyz="2.70300300277055E-11"
-                izz="0.664242254581203" />
-        </inertial>
-        <visual>
-            <origin xyz="0 0 0"
-                    rpy="0 0 0" />
-            <geometry>
-                <mesh filename="${mesh_location}/arm_gripper.stl" />
-            </geometry>
-            <material
-                name="">
-                <color rgba="1 1 1 1" />
-            </material>
-        </visual>
-        <collision>
-            <origin xyz="0 0 0"
-                    rpy="0 0 0" />
-            <geometry>
-                <mesh filename="${mesh_location}/arm_gripper.stl" />
-            </geometry>
-        </collision>
-    </link>
-    <joint name="arm_gripper_joint" type="revolute">
+    <!--Arm Wrist Link -->
+    <link name="arm_wrist_link">
+        <inertial>
+            <origin xyz="0 0 0" rpy="0 0 0" />
+            <mass value="1.5363204791731" />
+            <inertia
+                ixx="0.242660790998556"
+                ixy="-9.00009815481889E-05"
+                ixz="0.0234683038167963"
+                iyy="0.514730499629884"
+                iyz="2.70300300277055E-11"
+                izz="0.664242254581203" />
+        </inertial>
+        <visual>
+            <origin xyz="0 0 0"
+                    rpy="0 0 0" />
+            <geometry>
+                <mesh filename="${mesh_location}/arm_wrist.stl" />
+            </geometry>
+            <material
+                name="">
+                <color rgba="1 1 1 1" />
+            </material>
+        </visual>
+        <collision>
+            <origin xyz="0 0 0"
+                    rpy="0 0 0" />
+            <geometry>
+                <mesh filename="${mesh_location}/arm_wrist.stl" />
+            </geometry>
+        </collision>
+    </link>
+    <joint name="arm_wrist_joint" type="revolute">
         <parent link="arm_elbow_link"/>
-        <child link="arm_gripper_link"/>
+        <child link="arm_wrist_link"/>
         <origin xyz="0.0 0.0 0.4159" rpy="0.0 0.0 0.0"/>
         <axis xyz="1 0 0"/>
@@ -168,3 +169,124 @@
         <dynamics damping="10" friction="2"/>
     </joint>
+    <!--Arm gripper base Link -->
+    <link name="arm_gripper_base_link">
+        <inertial>
+            <origin xyz="0 0 0" rpy="0 0 0" />
+            <mass value="1.5363204791731" />
+            <inertia
+                ixx="0.242660790998556"
+                ixy="-9.00009815481889E-05"
+                ixz="0.0234683038167963"
+                iyy="0.514730499629884"
+                iyz="2.70300300277055E-11"
+                izz="0.664242254581203" />
+        </inertial>
+        <visual>
+            <origin xyz="0 0 0"
+                    rpy="0 0 0" />
+            <geometry>
+                <mesh filename="${mesh_location}/gripper_base.stl" />
+            </geometry>
+            <material
+                name="">
+                <color rgba="1 1 1 1" />
+            </material>
+        </visual>
+        <collision>
+            <origin xyz="0 0 0"
+                    rpy="0 0 0" />
+            <geometry>
+                <mesh filename="${mesh_location}/gripper_base.stl" />
+            </geometry>
+        </collision>
+    </link>
+    <joint name="arm_gripper_base_joint" type="revolute">
+        <parent link="arm_wrist_link"/>
+        <child link="arm_gripper_base_link"/>
+        <origin xyz="0.05655 0.0 0.1025" rpy="0.0 0.0 0.0"/>
+        <axis xyz="0 0 1"/>
+        <limit effort="500" velocity="1.0" lower="-1.57" upper="1.57"/>
+        <dynamics damping="10" friction="2"/>
+    </joint>
+    <!--Arm gripper left Link -->
+    <link name="arm_gripper_left_link">
+        <inertial>
+            <origin xyz="0 0 0" rpy="0 0 0" />
+            <mass value="1.5363204791731" />
+            <inertia
+                ixx="0.242660790998556"
+                ixy="-9.00009815481889E-05"
+                ixz="0.0234683038167963"
+                iyy="0.514730499629884"
+                iyz="2.70300300277055E-11"
+                izz="0.664242254581203" />
+        </inertial>
+        <visual>
+            <origin xyz="0 0 0"
+                    rpy="0 0 0" />
+            <geometry>
+                <mesh filename="${mesh_location}/gripper_left.stl" />
+            </geometry>
+            <material
+                name="">
+                <color rgba="1 1 1 1" />
+            </material>
+        </visual>
+        <collision>
+            <origin xyz="0 0 0"
+                    rpy="0 0 0" />
+            <geometry>
+                <mesh filename="${mesh_location}/gripper_left.stl" />
+            </geometry>
+        </collision>
+    </link>
+    <joint name="arm_gripper_left_joint" type="prismatic">
+        <parent link="arm_gripper_base_link"/>
+        <child link="arm_gripper_left_link"/>
+        <origin xyz="-0.1393 0.0 0.06453" rpy="0.0 0.0 0.0"/>
+        <axis xyz="1 0 0"/>
+        <limit effort="500" velocity="1.0" lower="0.0" upper="0.08925"/>
+        <dynamics damping="10" friction="2"/>
+    </joint>
+    <!--Arm gripper right Link -->
+    <link name="arm_gripper_right_link">
+        <inertial>
+            <origin xyz="0 0 0" rpy="0 0 0" />
+            <mass value="1.5363204791731" />
+            <inertia
+                ixx="0.242660790998556"
+                ixy="-9.00009815481889E-05"
+                ixz="0.0234683038167963"
+                iyy="0.514730499629884"
+                iyz="2.70300300277055E-11"
+                izz="0.664242254581203" />
+        </inertial>
+        <visual>
+            <origin xyz="0 0 0"
+                    rpy="0 0 0" />
+            <geometry>
+                <mesh filename="${mesh_location}/gripper_right.stl" />
+            </geometry>
+            <material
+                name="">
+                <color rgba="1 1 1 1" />
+            </material>
+        </visual>
+        <collision>
+            <origin xyz="0 0 0"
+                    rpy="0 0 0" />
+            <geometry>
+                <mesh filename="${mesh_location}/gripper_right.stl" />
+            </geometry>
+        </collision>
+    </link>
+    <joint name="arm_gripper_right_joint" type="prismatic">
+        <parent link="arm_gripper_base_link"/>
+        <child link="arm_gripper_right_link"/>
+        <origin xyz="0.1393 0.0 0.06453" rpy="0.0 0.0 0.0"/>
+        <axis xyz="-1 0 0"/>
+        <limit effort="500" velocity="1.0" lower="0.0" upper="0.08925"/>
+        <dynamics damping="10" friction="2"/>
+        <mimic joint="arm_gripper_left_joint" multiplier="1.0" offset="0.0"/>
+    </joint>
 </robot>

File: src/aries/urdf/common_properties.xacro (robot description, xacro)
@@ -23,4 +23,4 @@
     <xacro:property name="enable_lidar" value="false"/>
     <!-- Enable D435i -->
-    <xacro:property name="enable_D435i" value="true"/>
+    <xacro:property name="enable_D435i" value="false"/>
 </robot>

File: src/aries/urdf/left_link.xacro (robot description, xacro)
@@ -17,5 +17,5 @@
             <origin xyz="0 0 0" rpy="0 0 0"/>
             <geometry>
-                <mesh filename="${mesh_location}/R_Rocker_Link.STL"/>
+                <mesh filename="${mesh_location}/L_Rocker_Link.STL"/>
             </geometry>
             <material name="silver"/>
@@ -24,5 +24,5 @@
             <origin xyz="0 0 0" rpy="0 0 0"/>
             <geometry>
-                <mesh filename="${mesh_location}/R_Rocker_Link.STL"/>
+                <mesh filename="${mesh_location}/L_Rocker_Link.STL"/>
             </geometry>
         </collision>
@@ -53,5 +53,5 @@
             <origin xyz="0 0 0" rpy="0 0 0"/>
             <geometry>
-                <mesh filename="${mesh_location}/R_1_Wheel_Link.STL"/>
+                <mesh filename="${mesh_location}/L_1_Wheel_Link.STL"/>
             </geometry>
             <material name="blue"/>
@@ -88,5 +88,5 @@
             <origin xyz="0 0 0" rpy="0 0 0"/>
             <geometry>
-                <mesh filename="${mesh_location}/R_2_Wheel_Link.STL"/>
+                <mesh filename="${mesh_location}/L_2_Wheel_Link.STL"/>
             </geometry>
             <material name="blue"/>
@@ -123,5 +123,5 @@
             <origin xyz="0 0 0" rpy="0 0 0"/>
             <geometry>
-                <mesh filename="${mesh_location}/R_3_Wheel_Link.STL"/>
+                <mesh filename="${mesh_location}/L_3_Wheel_Link.STL"/>
             </geometry>
             <material name="blue"/>
@@ -158,5 +158,5 @@
             <origin xyz="0 0 0" rpy="0 0 0"/>
             <geometry>
-                <mesh filename="${mesh_location}/R_Boggie_Link.STL"/>
+                <mesh filename="${mesh_location}/L_Boggie_Link.STL"/>
             </geometry>
             <material name="silver"/>
@@ -165,5 +165,5 @@
             <origin xyz="0 0 0" rpy="0 0 0"/>
             <geometry>
-                <mesh filename="${mesh_location}/R_Boggie_Link.STL"/>
+                <mesh filename="${mesh_location}/L_Boggie_Link.STL"/>
             </geometry>
         </collision>
@@ -176,5 +176,5 @@
         <axis xyz="0 0 -1"/>
         <limit lower="-0.391" upper="0.527" effort="10" velocity="100"/>
-        <dynamics damping="0.01" friction="0.01"/>
+        <dynamics damping="50" friction="5"/>
     </joint>
     <link name="aux_L_Rocker_Link">

File: src/aries/urdf/right_link.xacro (robot description, xacro)
@@ -17,5 +17,5 @@
             <origin xyz="0 0 0" rpy="0 0 0"/>
             <geometry>
-                <mesh filename="${mesh_location}/L_Rocker_Link.STL"/>
+                <mesh filename="${mesh_location}/R_Rocker_Link.STL"/>
             </geometry>
             <material name="silver"/>
@@ -24,5 +24,5 @@
             <origin xyz="0 0 0" rpy="0 0 0"/>
             <geometry>
-                <mesh filename="${mesh_location}/L_Rocker_Link.STL"/>
+                <mesh filename="${mesh_location}/R_Rocker_Link.STL"/>
             </geometry>
         </collision>
@@ -34,5 +34,5 @@
         <child link="R_Rocker_Link"/>
         <axis xyz="0 0 -1"/>
-        <limit upper="-0.226" lower="0.323" effort="1000" velocity="5"/>
+        <limit upper="0.323" lower="-0.226" effort="1000" velocity="5"/>
         <xacro:if value="${enable_mimic}">
             <mimic joint="L_Rocker_Joint" multiplier="-1.0" offset="0.0"/>
@@ -56,5 +56,5 @@
             <origin xyz="0 0 0" rpy="0 0 0"/>
             <geometry>
-                <mesh filename="${mesh_location}/L_1_Wheel_Link.STL"/>
+                <mesh filename="${mesh_location}/R_1_Wheel_Link.STL"/>
             </geometry>
             <material name="blue"/>
@@ -91,5 +91,5 @@
             <origin xyz="0 0 0" rpy="0 0 0"/>
             <geometry>
-                <mesh filename="${mesh_location}/L_2_Wheel_Link.STL"/>
+                <mesh filename="${mesh_location}/R_2_Wheel_Link.STL"/>
             </geometry>
             <material name="blue"/>
@@ -126,5 +126,5 @@
             <origin xyz="0 0 0" rpy="0 0 0"/>
             <geometry>
-                <mesh filename="${mesh_location}/L_3_Wheel_Link.STL"/>
+                <mesh filename="${mesh_location}/R_3_Wheel_Link.STL"/>
             </geometry>
             <material name="blue"/>
@@ -161,5 +161,5 @@
             <origin xyz="0 0 0" rpy="0 0 0"/>
             <geometry>
-                <mesh filename="${mesh_location}/L_Boggie_Link.STL"/>
+                <mesh filename="${mesh_location}/R_Boggie_Link.STL"/>
             </geometry>
             <material name="silver"/>
@@ -168,5 +168,5 @@
             <origin xyz="0 0 0" rpy="0 0 0"/>
             <geometry>
-                <mesh filename="${mesh_location}/L_Boggie_Link.STL"/>
+                <mesh filename="${mesh_location}/R_Boggie_Link.STL"/>
             </geometry>
         </collision>
@@ -179,5 +179,5 @@
         <axis xyz="0 0 -1"/>
         <limit lower="-0.560" upper="0.594" effort="10" velocity="100"/>
-        <dynamics damping="0.01" friction="0.01"/>
+        <dynamics damping="50" friction="5"/>
     </joint>
     <link name="aux_R_Rocker_Link">

File: src/aries_moveit/config/aries.ros2_control.xacro (robot description, xacro)
@@ -10,5 +10,4 @@
             <joint name="arm_base_joint">
                 <command_interface name="position"/>
-                <command_interface name="velocity"/>
                 <state_interface name="position">
                   <param name="initial_value">${initial_positions['arm_base_joint']}</param>
@@ -18,5 +17,4 @@
             <joint name="arm_shoulder_joint">
                 <command_interface name="position"/>
-                <command_interface name="velocity"/>
                 <state_interface name="position">
                   <param name="initial_value">${initial_positions['arm_shoulder_joint']}</param>
@@ -26,5 +24,4 @@
             <joint name="arm_elbow_joint">
                 <command_interface name="position"/>
-                <command_interface name="velocity"/>
                 <state_interface name="position">
                   <param name="initial_value">${initial_positions['arm_elbow_joint']}</param>
@@ -32,9 +29,22 @@
                 <state_interface name="velocity"/>
             </joint>
-            <joint name="arm_gripper_joint">
+            <joint name="arm_wrist_joint">
                 <command_interface name="position"/>
-                <command_interface name="velocity"/>
                 <state_interface name="position">
-                  <param name="initial_value">${initial_positions['arm_gripper_joint']}</param>
+                  <param name="initial_value">${initial_positions['arm_wrist_joint']}</param>
+                </state_interface>
+                <state_interface name="velocity"/>
+            </joint>
+            <joint name="arm_gripper_base_joint">
+                <command_interface name="position"/>
+                <state_interface name="position">
+                  <param name="initial_value">${initial_positions['arm_gripper_base_joint']}</param>
+                </state_interface>
+                <state_interface name="velocity"/>
+            </joint>
+            <joint name="arm_gripper_left_joint">
+                <command_interface name="position"/>
+                <state_interface name="position">
+                  <param name="initial_value">${initial_positions['arm_gripper_left_joint']}</param>
                 </state_interface>
                 <state_interface name="velocity"/>
