Commit message: commit

File: src/aries/urdf/aries_gazebo.xacro (robot description, xacro)
@@ -110,11 +110,10 @@
             filename="gz-sim-joint-state-publisher-system"
             name="gz::sim::systems::JointStatePublisher">
-            <joint_name>arm_base_joint</joint_name>
-            <joint_name>arm_shoulder_joint</joint_name>
-            <joint_name>arm_elbow_joint</joint_name>
-            <joint_name>arm_wrist_joint</joint_name>
-            <joint_name>arm_gripper_base_joint</joint_name>
-            <joint_name>arm_gripper_left_joint</joint_name>
-            <joint_name>arm_gripper_right_joint</joint_name>
+            <joint_name>joint1</joint_name>
+            <joint_name>joint2</joint_name>
+            <joint_name>joint3</joint_name>
+            <joint_name>joint4</joint_name>
+            <joint_name>joint5</joint_name>
+            <joint_name>joint6</joint_name>
             <joint_name>L_Rocker_Joint</joint_name>
             <joint_name>R_Rocker_Joint</joint_name>
@@ -160,6 +159,6 @@
     <plugin filename="gz-sim-joint-position-controller-system"
         name="gz::sim::systems::JointPositionController">
-      <joint_name>arm_base_joint</joint_name>
-      <topic>/model/aries/joint/arm_base_joint/cmd_pos</topic>
+      <joint_name>joint1</joint_name>
+      <topic>/model/aries/joint/joint1/cmd_pos</topic>
       <initial_position>0.0</initial_position>
       <p_gain>300</p_gain><i_gain>2</i_gain><d_gain>30</d_gain>
@@ -168,6 +167,6 @@
     <plugin filename="gz-sim-joint-position-controller-system"
         name="gz::sim::systems::JointPositionController">
-      <joint_name>arm_shoulder_joint</joint_name>
-      <topic>/model/aries/joint/arm_shoulder_joint/cmd_pos</topic>
+      <joint_name>joint2</joint_name>
+      <topic>/model/aries/joint/joint2/cmd_pos</topic>
       <initial_position>0.510</initial_position>
       <p_gain>300</p_gain><i_gain>2</i_gain><d_gain>30</d_gain>
@@ -176,6 +175,6 @@
     <plugin filename="gz-sim-joint-position-controller-system"
         name="gz::sim::systems::JointPositionController">
-      <joint_name>arm_elbow_joint</joint_name>
-      <topic>/model/aries/joint/arm_elbow_joint/cmd_pos</topic>
+      <joint_name>joint3</joint_name>
+      <topic>/model/aries/joint/joint3/cmd_pos</topic>
       <initial_position>1.748</initial_position>
       <p_gain>300</p_gain><i_gain>2</i_gain><d_gain>30</d_gain>
@@ -184,6 +183,6 @@
     <plugin filename="gz-sim-joint-position-controller-system"
         name="gz::sim::systems::JointPositionController">
-      <joint_name>arm_wrist_joint</joint_name>
-      <topic>/model/aries/joint/arm_wrist_joint/cmd_pos</topic>
+      <joint_name>joint4</joint_name>
+      <topic>/model/aries/joint/joint4/cmd_pos</topic>
       <initial_position>1.420</initial_position>
       <p_gain>300</p_gain><i_gain>2</i_gain><d_gain>30</d_gain>
@@ -192,6 +191,6 @@
     <plugin filename="gz-sim-joint-position-controller-system"
         name="gz::sim::systems::JointPositionController">
-      <joint_name>arm_gripper_base_joint</joint_name>
-      <topic>/model/aries/joint/arm_gripper_base_joint/cmd_pos</topic>
+      <joint_name>joint5</joint_name>
+      <topic>/model/aries/joint/joint5/cmd_pos</topic>
       <initial_position>0.0</initial_position>
       <p_gain>300</p_gain><i_gain>2</i_gain><d_gain>30</d_gain>
@@ -200,14 +199,6 @@
     <plugin filename="gz-sim-joint-position-controller-system"
         name="gz::sim::systems::JointPositionController">
-      <joint_name>arm_gripper_left_joint</joint_name>
-      <topic>/model/aries/joint/arm_gripper_left_joint/cmd_pos</topic>
-      <initial_position>0.0</initial_position>
-      <p_gain>300</p_gain><i_gain>2</i_gain><d_gain>30</d_gain>
-      <i_min>-6</i_min><i_max>6</i_max>
-    </plugin>
-    <plugin filename="gz-sim-joint-position-controller-system"
-        name="gz::sim::systems::JointPositionController">
-      <joint_name>arm_gripper_right_joint</joint_name>
-      <topic>/model/aries/joint/arm_gripper_right_joint/cmd_pos</topic>
+      <joint_name>joint6</joint_name>
+      <topic>/model/aries/joint/joint6/cmd_pos</topic>
       <initial_position>0.0</initial_position>
       <p_gain>300</p_gain><i_gain>2</i_gain><d_gain>30</d_gain>

File: src/aries/urdf/common_properties.xacro (robot description, xacro)
@@ -21,6 +21,6 @@
     <xacro:property name="enable_mimic" value="true"/>
     <!-- Enable Lidar -->
-    <xacro:property name="enable_lidar" value="false"/>
+    <xacro:property name="enable_lidar" value="true"/>
     <!-- Enable D435i -->
-    <xacro:property name="enable_D435i" value="false"/>
+    <xacro:property name="enable_D435i" value="true"/>
 </robot>

File: src/aries/urdf/my_robot.urdf.xacro (robot description, xacro)
@@ -2,12 +2,14 @@
 <robot name="aries" xmlns:xacro="http://www.ros.org/wiki/xacro">
     <xacro:include filename="common_properties.xacro" />
-    <xacro:include filename="aries_gazebo.xacro" />
+    <!-- <xacro:include filename="aries_gazebo.xacro" />
     <xacro:include filename="aries_base.xacro" />
     <xacro:include filename="differential_link.xacro" />
     <xacro:include filename="left_link.xacro" />
     <xacro:include filename="right_link.xacro" />
-    <xacro:include filename="lidar.xacro" />
+    <xacro:include filename="lidar.xacro" /> -->
     <!-- <xacro:include filename="camera.xacro" /> -->
-    <xacro:include filename="d435i.xacro" />
-    <xacro:include filename="arm.xacro" />
+    <!-- <xacro:include filename="d435i.xacro" /> -->
+    <!-- <xacro:include filename="arm.xacro" /> -->
+    <!-- <xacro:include filename="igus_rebel_robot2.urdf.xacro" /> -->
+    <xacro:include filename="gripper_new.xacro" />
 </robot>

Commit message: commit

File: src/aries/urdf/aries_gazebo.xacro (robot description, xacro)
@@ -116,4 +116,10 @@
             <joint_name>joint5</joint_name>
             <joint_name>joint6</joint_name>
+            <joint_name>gripper_gear_left_joint</joint_name>
+            <joint_name>gripper_gear_right_joint</joint_name>
+            <joint_name>gripper_link_left_joint</joint_name>
+            <joint_name>gripper_link_right_joint</joint_name>
+            <joint_name>gripper_bucket_right_joint</joint_name>
+            <joint_name>gripper_bucket_left_joint</joint_name>
             <joint_name>L_Rocker_Joint</joint_name>
             <joint_name>R_Rocker_Joint</joint_name>
@@ -162,5 +168,5 @@
       <topic>/model/aries/joint/joint1/cmd_pos</topic>
       <initial_position>0.0</initial_position>
-      <p_gain>300</p_gain><i_gain>2</i_gain><d_gain>30</d_gain>
+      <p_gain>1000</p_gain><i_gain>2</i_gain><d_gain>300</d_gain>
       <i_min>-6</i_min><i_max>6</i_max>
     </plugin>
@@ -170,5 +176,5 @@
       <topic>/model/aries/joint/joint2/cmd_pos</topic>
       <initial_position>0.510</initial_position>
-      <p_gain>300</p_gain><i_gain>2</i_gain><d_gain>30</d_gain>
+      <p_gain>1000</p_gain><i_gain>2</i_gain><d_gain>300</d_gain>
       <i_min>-6</i_min><i_max>6</i_max>
     </plugin>
@@ -178,5 +184,5 @@
       <topic>/model/aries/joint/joint3/cmd_pos</topic>
       <initial_position>1.748</initial_position>
-      <p_gain>300</p_gain><i_gain>2</i_gain><d_gain>30</d_gain>
+      <p_gain>1000</p_gain><i_gain>2</i_gain><d_gain>300</d_gain>
       <i_min>-6</i_min><i_max>6</i_max>
     </plugin>
@@ -186,5 +192,5 @@
       <topic>/model/aries/joint/joint4/cmd_pos</topic>
       <initial_position>1.420</initial_position>
-      <p_gain>300</p_gain><i_gain>2</i_gain><d_gain>30</d_gain>
+      <p_gain>1000</p_gain><i_gain>2</i_gain><d_gain>300</d_gain>
       <i_min>-6</i_min><i_max>6</i_max>
     </plugin>
@@ -194,5 +200,5 @@
       <topic>/model/aries/joint/joint5/cmd_pos</topic>
       <initial_position>0.0</initial_position>
-      <p_gain>300</p_gain><i_gain>2</i_gain><d_gain>30</d_gain>
+      <p_gain>1000</p_gain><i_gain>2</i_gain><d_gain>300</d_gain>
       <i_min>-6</i_min><i_max>6</i_max>
     </plugin>
@@ -201,6 +207,14 @@
       <joint_name>joint6</joint_name>
       <topic>/model/aries/joint/joint6/cmd_pos</topic>
+      <initial_position>0.523599</initial_position>
+      <p_gain>1000</p_gain><i_gain>2</i_gain><d_gain>300</d_gain>
+      <i_min>-6</i_min><i_max>6</i_max>
+    </plugin>
+    <plugin filename="gz-sim-joint-position-controller-system"
+        name="gz::sim::systems::JointPositionController">
+      <joint_name>gripper_gear_left_joint</joint_name>
+      <topic>/model/aries/joint/gripper_gear_left_joint/cmd_pos</topic>
       <initial_position>0.0</initial_position>
-      <p_gain>300</p_gain><i_gain>2</i_gain><d_gain>30</d_gain>
+      <p_gain>1000</p_gain><i_gain>2</i_gain><d_gain>300</d_gain>
       <i_min>-6</i_min><i_max>6</i_max>
     </plugin>

File: src/aries/urdf/gripper_new.xacro (robot description, xacro)
@@ -1,4 +1,9 @@
 <?xml version="1.0"?>
 <robot xmlns:xacro="http://www.ros.org/wiki/xacro">
+    <joint name="arm_gripper_base_joint" type="fixed">
+        <parent link="link6"/>
+        <child link="gripper_base_link"/>
+        <origin xyz="0.0 0.0 0.05223" rpy="0.0 0.0 0.523599"/>
+    </joint>
     <!--gripper base Link -->
     <link name="gripper_base_link">

File: src/aries/urdf/my_robot.urdf.xacro (robot description, xacro)
@@ -2,14 +2,14 @@
 <robot name="aries" xmlns:xacro="http://www.ros.org/wiki/xacro">
     <xacro:include filename="common_properties.xacro" />
-    <!-- <xacro:include filename="aries_gazebo.xacro" />
+    <xacro:include filename="aries_gazebo.xacro" />
     <xacro:include filename="aries_base.xacro" />
     <xacro:include filename="differential_link.xacro" />
     <xacro:include filename="left_link.xacro" />
     <xacro:include filename="right_link.xacro" />
-    <xacro:include filename="lidar.xacro" /> -->
+    <xacro:include filename="lidar.xacro" />
     <!-- <xacro:include filename="camera.xacro" /> -->
-    <!-- <xacro:include filename="d435i.xacro" /> -->
+    <xacro:include filename="d435i.xacro" />
     <!-- <xacro:include filename="arm.xacro" /> -->
-    <!-- <xacro:include filename="igus_rebel_robot2.urdf.xacro" /> -->
+    <xacro:include filename="igus_rebel_robot2.urdf.xacro" />
     <xacro:include filename="gripper_new.xacro" />
 </robot>

Commit message: Initial commit: aries_autonomy ROS 2 workspace

File: src/aries/urdf/aries_gazebo.xacro (robot description, xacro)
@@ -241,5 +241,7 @@
         </plugin>
   </gazebo>
+  <!-- IMU Plugin
   <gazebo reference="imu_frame">
+      <plugin filename='gz-sim-imu-system' name='gz::sim::systems::Imu'/>
       <sensor name="imu_sensor" type="imu">
           <always_on>1</always_on>
@@ -249,4 +251,27 @@
           <topic>/imu</topic>
       </sensor>
+  </gazebo> -->
+  <!-- IMU Sensor -->
+  <gazebo reference="imu_frame">
+    <sensor name="imu_sensor" type="imu">
+      <always_on>true</always_on>
+      <update_rate>60</update_rate>
+      <visualize>true</visualize>
+      <topic>/imu</topic>
+      <imu>
+        <angular_velocity>
+          <x>0</x>
+          <y>0</y>
+          <z>0</z>
+        </angular_velocity>
+        <linear_acceleration>
+          <x>0</x>
+          <y>0</y>
+          <z>0</z>
+        </linear_acceleration>
+      </imu>
+      <plugin filename="gz-sim-imu-system"
+              name="gz::sim::systems::Imu"/>
+    </sensor>
   </gazebo>
   <!-- Gazebo Plugin for Diff Drive -->

File: src/aries/urdf/common_properties.xacro (robot description, xacro)
@@ -17,9 +17,9 @@
     <xacro:property name="wheel_thickness" value="0.070"/>
     <!-- Mesh locations -->
-    <xacro:property name="mesh_location" value="file:///home/shreyas/aries/src/aries/meshes"/>
+    <xacro:property name="mesh_location" value="file:///home/rahul/aries_autonomy/src/aries/meshes"/>
     <!-- Enable Mimic joints -->
     <xacro:property name="enable_mimic" value="true"/>
     <!-- Enable Lidar -->
-    <xacro:property name="enable_lidar" value="true"/>
+    <xacro:property name="enable_lidar" value="false"/>
     <!-- Enable D435i -->
     <xacro:property name="enable_D435i" value="true"/>
